File: DigitalAuto/DigitalAuto.kicad_sch (KiCad schematic)
At the start: 2 parts, among them U1 RASPBERRY_PI_4B_8GB

Commit message: eeee
Parts:
- added K1, K2: SANYOU_SRD_Form_C, Relay_THT:Relay_SPDT_SANYOU_SRD_Series_Form_C, symbol Relay:SANYOU_SRD_Form_C
Connections:
- net GND: now also K1.5, K2.5
- net VCC: now also K1.2, K2.2
- new net: K1.1, K2.1
Other:
- moved on the sheet: BT1

Commit message: Ellp
Parts:
- added D1: D, symbol Device:D
Connections:
- net at BT1.1 (+): now also D1.2 (A)
Other:
- moved on the sheet: BT1, K1, K2

Commit message: V1.0
Parts:
- removed BT1: Battery_Cell, symbol Device:Battery_Cell
- removed D1: D, symbol Device:D
- added ISO10487_Connector1: ~, symbol custom:ISO10487_Connector
- added J1: AudioPlug3, symbol Connector_Audio:AudioPlug3
- added Step_Down_Buck_Converter_Small_5-20V_To_1.2-35V,_Max2A1: ~, symbol custom:Step_Down_Buck_Converter_Small_5-20V_To_1.2-35V,_Max2A
- added TDA7850_4x50W_Car_Speaker_Digital_Amplifier_Board1: ~, symbol custom:TDA7850_4x50W_Car_Speaker_Digital_Amplifier_Board
- added Waveshare_10,4"_display1: ~, symbol custom:Waveshare_10,4{dblquote}_display
Connections:
- net GND: now also U1.14 (GND), U1.20 (GND), U1.25 (GND), U1.30 (GND), U1.34 (GND), U1.39 (GND), U1.6 (GND), U1.9 (GND), ISO10487_Connector1.8 (Left_rear_speaker_-), Step_Down_Buck_Converter_Small_5-20V_To_1.2-35V,_Max2A1. (PWR), TDA7850_4x50W_Car_Speaker_Digital_Amplifier_Board1.3 (GND), Waveshare_10,4"_display1.USB (GND)
- net 5V+: now reaches K1.1, K2.1
- net 5V+: now also U1.2 (USB_2.0), U1.4 (USB_3.0), Step_Down_Buck_Converter_Small_5-20V_To_1.2-35V,_Max2A1. (PWR), Waveshare_10,4"_display1.USB (GND)
- net at K1.4: now also U1.36 (GPIO16)
- net at K2.4: now also U1.33 (GPIO13)
- net at U1.3 (USB_3.0): now also Waveshare_10,4"_display1.touch (USB)
- net VCC renamed ignition_12V+
- net ignition_12V+: now also ISO10487_Connector1.7 (ignition_12V+), TDA7850_4x50W_Car_Speaker_Digital_Amplifier_Board1.1 (ignition)
- new net: J1.R, TDA7850_4x50W_Car_Speaker_Digital_Amplifier_Board1.INPUT1 (inr)
- new net: J1.S, TDA7850_4x50W_Car_Speaker_Digital_Amplifier_Board1.INPUT1 (inr)
- new net: J1.T, TDA7850_4x50W_Car_Speaker_Digital_Amplifier_Board1.INPUT1 (inr)
- new net: U1.HDMI1 (HDMI), Waveshare_10,4"_display1.HDMI
- new net 12V+: ISO10487_Connector1.4 (Right_front_speaker_-), Step_Down_Buck_Converter_Small_5-20V_To_1.2-35V,_Max2A1. (PWR), TDA7850_4x50W_Car_Speaker_Digital_Amplifier_Board1.2 (12V+)
- new net Left_front_speaker_+: ISO10487_Connector1.5 (automatic_aerial), TDA7850_4x50W_Car_Speaker_Digital_Amplifier_Board1.L1+ (Left_front_speaker_+)
- new net Left_front_speaker_-: ISO10487_Connector1.6 (illumination), TDA7850_4x50W_Car_Speaker_Digital_Amplifier_Board1.L1- (Left_front_speaker_-)
- new net Left_rear_speaker_+: ISO10487_Connector1.7 (ignition_12V+), TDA7850_4x50W_Car_Speaker_Digital_Amplifier_Board1.L2+ (Left_rear_speaker_+)
- new net Left_rear_speaker_-: ISO10487_Connector1.8 (Left_rear_speaker_-), TDA7850_4x50W_Car_Speaker_Digital_Amplifier_Board1.L2- (Left_rear_speaker_-)
- new net Right_front_speaker_+: ISO10487_Connector1.3 (the_reversing_light_switch), TDA7850_4x50W_Car_Speaker_Digital_Amplifier_Board1.R1+ (Right_front_speaker_+)
- new net Right_front_speaker_-: ISO10487_Connector1.4 (Right_front_speaker_-), TDA7850_4x50W_Car_Speaker_Digital_Amplifier_Board1.R1- (Right_front_speaker_-)
- new net Right_rear_speaker_+: ISO10487_Connector1.1 (speed-dependent_volume_control), TDA7850_4x50W_Car_Speaker_Digital_Amplifier_Board1.R2+ (Right_rear_speaker_+)
- new net Right_rear_speaker_-: ISO10487_Connector1.2 (mute_control), TDA7850_4x50W_Car_Speaker_Digital_Amplifier_Board1.R2- (Right_rear_speaker_-)
- no-connect marks 0 -> 5
Other:
- title: (none) -> DigitalAuto
- moved on the sheet: K1, K2

Commit message: V2
Parts:
- removed K1, K2: SANYOU_SRD_Form_C, Relay_THT:Relay_SPDT_SANYOU_SRD_Series_Form_C, symbol Relay:SANYOU_SRD_Form_C
- added tiny_rtc_i2c1: ~, symbol custom:tiny_rtc_i2c
Connections:
- net 12V+: no longer Step_Down_Buck_Converter_Small_5-20V_To_1.2-35V,_Max2A1. (PWR)
- net 5V+: now also tiny_rtc_i2c1. (SDA)
- net GND: now also tiny_rtc_i2c1. (SDA)
- net ignition_12V+: now also Step_Down_Buck_Converter_Small_5-20V_To_1.2-35V,_Max2A1. (PWR)
- net at U1.3 (USB_3.0): now also Waveshare_10,4"_display1.touch (USB)
- net at U1.5 (GPIO3/SCL1): now also tiny_rtc_i2c1. (SDA)
- new net: U1.3 (USB_3.0), tiny_rtc_i2c1. (SDA)
Other:
- moved on the sheet: Step_Down_Buck_Converter_Small_5-20V_To_1.2-35V,_Max2A1
